File: v1.3/RAMPSdisplay.brd (EAGLE design)
At the start: 141.6 x 72.4 mm, 35 parts, among them IC1 LD1117, IC2 HEF4050B, IC3 MAX31855K, IC4 MAX31855K, IC5 MAX31855K, J1 PCC-SMP-V-K, J2 PCC-SMP-V-K, J3 Micro-SD socket, J4 Interface, J5 PCC-SMP-V-K, Q1 2N7002, Q2 Piezo, SW1 CI-11

Commit message: foo
Routing:
- net SW: track 54.8 -> 55.4 mm
Changed lines of the file:
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@@
 <contactref element="J4" pad="8"/>
 <wire x1="135.89" y1="22.225" x2="134.62" y2="23.495" width="0.4064" layer="16"/>
-<wire x1="134.62" y1="23.495" x2="126.365" y2="23.495" width="0.4064" layer="16"/>
-<wire x1="124.46" y1="25.4" x2="126.365" y2="23.495" width="0.4064" layer="16"/>
-<wire x1="99.06" y1="25.4" x2="124.46" y2="25.4" width="0.6096" layer="16"/>
+<wire x1="134.62" y1="23.495" x2="128.27" y2="23.495" width="0.4064" layer="16"/>
+<wire x1="126.365" y1="25.4" x2="128.27" y2="23.495" width="0.4064" layer="16"/>
+<wire x1="99.06" y1="25.4" x2="126.365" y2="25.4" width="0.6096" layer="16"/>
 <wire x1="99.06" y1="25.4" x2="88.9" y2="35.56" width="0.6096" layer="16"/>
 </signal>
@@
 <wire x1="119.38" y1="12.065" x2="113.665" y2="12.065" width="0.4064" layer="1"/>
 <wire x1="113.665" y1="12.065" x2="111.125" y2="14.605" width="0.4064" layer="1"/>
-<wire x1="113.705" y1="29.86" x2="113.705" y2="26.035" width="0.4064" layer="1"/>
 <wire x1="133.35" y1="22.225" x2="129.54" y2="22.225" width="0.4064" layer="1"/>
 <wire x1="129.54" y1="22.225" x2="125.095" y2="26.67" width="0.4064" layer="1"/>
-<wire x1="115.61" y1="24.13" x2="113.705" y2="26.035" width="0.4064" layer="1"/>
-<wire x1="111.125" y1="19.645" x2="115.61" y2="24.13" width="0.4064" layer="1"/>
-<wire x1="111.125" y1="14.605" x2="111.125" y2="19.645" width="0.4064" layer="1"/>
-<wire x1="125.095" y1="26.67" x2="118.15" y2="26.67" width="0.4064" layer="1"/>
-<wire x1="118.15" y1="26.67" x2="115.61" y2="24.13" width="0.4064" layer="1"/>
+<wire x1="125.095" y1="26.67" x2="116.895" y2="26.67" width="0.4064" layer="1"/>
+<wire x1="116.895" y1="26.67" x2="113.705" y2="29.86" width="0.4064" layer="1"/>
+<wire x1="111.125" y1="14.605" x2="111.125" y2="17.145" width="0.4064" layer="1"/>
+<wire x1="111.125" y1="17.145" x2="113.665" y2="19.685" width="0.4064" layer="1"/>
+<wire x1="113.665" y1="19.685" x2="113.665" y2="29.82" width="0.4064" layer="1"/>
+<wire x1="113.665" y1="29.82" x2="113.705" y2="29.86" width="0.4064" layer="1"/>
 </signal>
 <signal name="B">
